File: sch/robot_controller.kicad_pcb (KiCad board)
At the start: 2 copper layers, 100 x 90 mm, 119 parts, among them IC1 ADM3058EBRIZ-RL, IC2 ADM3058EBRIZ-RL, IC3 74LVC2G125DP,125, IC4 74LVC2G125DP,125, IC5 ADM3058EBRIZ-RL, J1 USB_C_Receptacle_USB2.0, J10 Conn_01x03, J11 Conn_01x03, J12 Conn_01x03, J13 Conn_01x04, J14 Conn_01x04, J15 Conn_01x04, J16 Conn_01x02, J17 Conn_01x04, J18 Conn_01x04, J19 Conn_01x03, J2 Conn_01x06, J20 Conn_01x02, J21 Conn_01x03, J22 Conn_01x02, J23 Conn_02x03_Odd_Even, J3 RJ45_LED, J4 Conn_01x06, J5 Conn_01x03, J6 Conn_01x03, J7 Conn_01x03, J8 Conn_01x03, J9 Conn_01x03, Q1 2SC4116, Q2 2SC4116, Q3 IRLML6402, Q4 IRLML6402, U1 Teensy4.1_simple, U2 AZ1117-3.3, U3 ISO1540, U4 NCP718xSN500, U5 LD1117S50TR_SOT223

Commit message: fix : sch
Parts:
- moved Q3 0.59 mm to (110.0, 136.0), turned to 90 degrees
- turned Q4 to 0 degrees
Connections:
- Q3 pad 2: /ENC_VCC -> +5VP
- Q3 pad 3: +5VP -> /ENC_VCC
- Q4 pad 2: /WALL_VCC -> +5VP
- Q4 pad 3: +5VP -> /WALL_VCC
Routing:
- net Net-(Q1-Pad3): track 3.46 -> 6.75 mm
- net Net-(Q2-Pad3): track 3.91 -> 7.15 mm
- net /WALL_VCC: track 63.1 -> 64.0 mm
- net /ENC_VCC: track 17.0 -> 17.8 mm
Changed lines of the file:
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@@
     (thickness 1.6)
     (drawings 38)
-    (tracks 1152)
+    (tracks 1166)
     (zones 0)
     (modules 119)
@@
   (page A3)
   (layers
-    (0 F.Cu signal)
-    (31 B.Cu signal)
+    (0 F.Cu signal hide)
+    (31 B.Cu signal hide)
     (32 B.Adhes user)
     (33 F.Adhes user)
@@
   )
   (setup
-    (last_trace_width 0.25)
+    (last_trace_width 0.3)
     (user_trace_width 0.2)
     (user_trace_width 0.3)
@@
   )
   (module Package_TO_SOT_SMD:SOT-23 (layer F.Cu)
-    (at 110.575 136.125 270)
+    (at 110 136 90)
     (descr "SOT-23, Standard")
     (tags SOT-23)
@@
       (effects (font (size 0.5 0.5) (thickness 0.075)))
     )
-    (pad 3 smd rect (at 1 0 270) (size 0.9 0.8) (layers F.Cu F.Paste F.Mask)
-      (net 4 +5VP))
-    (pad 2 smd rect (at -1 0.95 270) (size 0.9 0.8) (layers F.Cu F.Paste F.Mask)
+    (pad 3 smd rect (at 1 0 90) (size 0.9 0.8) (layers F.Cu F.Paste F.Mask)
       (net 14 /ENC_VCC))
-    (pad 1 smd rect (at -1 -0.95 270) (size 0.9 0.8) (layers F.Cu F.Paste F.Mask)
+    (pad 2 smd rect (at -1 0.95 90) (size 0.9 0.8) (layers F.Cu F.Paste F.Mask)
+      (net 4 +5VP))
+    (pad 1 smd rect (at -1 -0.95 90) (size 0.9 0.8) (layers F.Cu F.Paste F.Mask)
       (net 74 "Net-(Q1-Pad3)"))
     (model ${KISYS3DMOD}/Package_TO_SOT_SMD.3dshapes/SOT-23.wrl
@@
   )
   (module Package_TO_SOT_SMD:SOT-23 (layer F.Cu)
-    (at 182.8 159.7 180)
+    (at 182.8 159.7)
     (descr "SOT-23, Standard")
     (tags SOT-23)
@@
     (fp_line (start 0.76 -1.58) (end -1.4 -1.58) (layer F.SilkS) (width 0.12))
     (fp_line (start 0.76 1.58) (end -0.7 1.58) (layer F.SilkS) (width 0.12))
-    (pad 1 smd rect (at -1 -0.95 180) (size 0.9 0.8) (layers F.Cu F.Paste F.Mask)
+    (pad 1 smd rect (at -1 -0.95) (size 0.9 0.8) (layers F.Cu F.Paste F.Mask)
       (net 77 "Net-(Q2-Pad3)"))
-    (pad 2 smd rect (at -1 0.95 180) (size 0.9 0.8) (layers F.Cu F.Paste F.Mask)
-      (net 17 /WALL_VCC))
-    (pad 3 smd rect (at 1 0 180) (size 0.9 0.8) (layers F.Cu F.Paste F.Mask)
+    (pad 2 smd rect (at -1 0.95) (size 0.9 0.8) (layers F.Cu F.Paste F.Mask)
       (net 4 +5VP))
+    (pad 3 smd rect (at 1 0) (size 0.9 0.8) (layers F.Cu F.Paste F.Mask)
+      (net 17 /WALL_VCC))
     (model ${KISYS3DMOD}/Package_TO_SOT_SMD.3dshapes/SOT-23.wrl
       (at (xyz 0 0 0))
@@
     (effects (font (size 0.7 0.7) (thickness 0.1)))
   )
-  (gr_text "Tnsy 5VL" (at 113.2 109.6 90) (layer F.SilkS)
+  (gr_text "Tnsy 5VL" (at 114.725 109.525 90) (layer F.SilkS)
     (effects (font (size 0.8 0.8) (thickness 0.15)))
   )
-  (gr_text "Ext 5VL" (at 114.7 109.2 90) (layer F.SilkS)
+  (gr_text "Ext 5VL" (at 113.25 109.15 90) (layer F.SilkS)
     (effects (font (size 0.8 0.8) (thickness 0.15)))
   )
-  (gr_text "Ext 5VP" (at 116.2 109.1 90) (layer F.SilkS)
+  (gr_text "Ext 5VP" (at 117.7 109.1 90) (layer F.SilkS)
     (effects (font (size 0.8 0.8) (thickness 0.15)))
   )
-  (gr_text "Tnsy 5VP" (at 117.7 109.5 90) (layer F.SilkS)
+  (gr_text "Tnsy 5VP" (at 116.2 109.475 90) (layer F.SilkS)
     (effects (font (size 0.8 0.8) (thickness 0.15)))
   )
@@
   (segment (start 117.255 155.2) (end 117.3 155.245) (width 0.3) (layer F.Cu) (net 2))
   (segment (start 117.255 154.425) (end 117.255 155.2) (width 0.3) (layer F.Cu) (net 2))
-  (via (at 111.9 137.5) (size 0.8) (drill 0.4) (layers F.Cu B.Cu) (net 2))
+  (via (at 112 137.9) (size 0.8) (drill 0.4) (layers F.Cu B.Cu) (net 2))
   (via (at 115.9 136) (size 0.8) (drill 0.4) (layers F.Cu B.Cu) (net 2))
   (via (at 112.9 140.9) (size 0.8) (drill 0.4) (layers F.Cu B.Cu) (net 2))
@@
   (segment (start 114.5 166) (end 113.995 166.505) (width 0.5) (layer F.Cu) (net 12))
   (segment (start 107.4 109.4) (end 105.77 109.4) (width 0.5) (layer F.Cu) (net 13))
-  (segment (start 106.7 138.05) (end 109.625 135.125) (width 0.5) (layer F.Cu) (net 14))
   (segment (start 106.5875 138.05) (end 106.7 138.05) (width 0.5) (layer F.Cu) (net 14))
-  (segment (start 109.625 133.875) (end 108.6 132.85) (width 0.8) (layer F.Cu) (net 14))
-  (segment (start 109.625 135.125) (end 109.625 133.875) (width 0.8) (layer F.Cu) (net 14))
-  (segment (start 108.6 132.85) (end 108.6 129.7) (width 0.8) (layer F.Cu) (net 14))
   (segment (start 108.6 122.8) (end 108.6 129.7) (width 0.8) (layer B.Cu) (net 14))
+  (segment (start 110 134.25) (end 110 135) (width 0.8) (layer F.Cu) (net 14))
+  (segment (start 108.6 129.7) (end 108.6 132.85) (width 0.8) (layer F.Cu) (net 14))
+  (segment (start 108.6 132.85) (end 110 134.25) (width 0.8) (layer F.Cu) (net 14))
+  (segment (start 109.3 135) (end 110 135) (width 0.3) (layer F.Cu) (net 14))
+  (segment (start 106.5875 137.575) (end 109.1625 135) (width 0.3) (layer F.Cu) (net 14))
+  (segment (start 109.1625 135) (end 109.3 135) (width 0.3) (layer F.Cu) (net 14))
+  (segment (start 106.5875 138.05) (end 106.5875 137.575) (width 0.3) (layer F.Cu) (net 14))
   (segment (start 103.585 138.05) (end 105.0125 138.05) (width 0.5) (layer F.Cu) (net 15))
   (segment (start 194.9875 159.2) (end 196.43 159.2) (width 0.3) (layer F.Cu) (net 16))
   (segment (start 183.8 157.35) (end 184.6 156.55) (width 1) (layer F.Cu) (net 17))
-  (segment (start 183.8 158.75) (end 183.8 157.35) (width 1) (layer F.Cu) (net 17))
   (segment (start 184.6 156.55) (end 184.6 153.5) (width 1) (layer F.Cu) (net 17))
   (segment (start 195.125 156.55) (end 196.2 155.475) (width 1) (layer F.Cu) (net 17))
@@
   (segment (start 196.2 146.7) (end 196.2 153.5) (width 1) (layer B.Cu) (net 17))
   (segment (start 196.2 155.475) (end 196.2 153.5) (width 1) (layer F.Cu) (net 17))
+  (segment (start 183.8 158.75) (end 183.8 157.35) (width 1) (layer F.Cu) (net 17))
+  (segment (start 183.8 158.75) (end 183.8 159.7) (width 1) (layer F.Cu) (net 17))
   (segment (start 107.4 111.9) (end 105.785 111.9) (width 0.5) (layer F.Cu) (net 18))
   (segment (start 169.6 180.95) (end 168.15 179.5) (width 0.5) (layer F.Cu) (net 19))
@@
   (segment (start 109 183.7) (end 109 184.9) (width 0.5) (layer F.Cu) (net 73))
   (segment (start 112.96 135.125) (end 112.975 135.14) (width 0.5) (layer F.Cu) (net 74))
-  (segment (start 111.525 135.125) (end 112.96 135.125) (width 0.5) (layer F.Cu) (net 74))
   (segment (start 112.99 135.125) (end 112.975 135.14) (width 0.5) (layer F.Cu) (net 74))
   (segment (start 114.975 135.125) (end 112.99 135.125) (width 0.5) (layer F.Cu) (net 74))
+  (segment (start 109.05 136.95) (end 109.05 137) (width 0.3) (layer F.Cu) (net 74))
+  (segment (start 109.75 136.25) (end 109.05 136.95) (width 0.3) (layer F.Cu) (net 74))
+  (segment (start 110.230002 136.25) (end 109.75 136.25) (width 0.3) (layer F.Cu) (net 74))
+  (segment (start 111.340002 135.14) (end 110.230002 136.25) (width 0.3) (layer F.Cu) (net 74))
+  (segment (start 112.975 135.14) (end 111.340002 135.14) (width 0.3) (layer F.Cu) (net 74))
   (segment (start 113.165 137.125) (end 113.025 137.265) (width 0.5) (layer F.Cu) (net 75))
   (segment (start 114.325 137.125) (end 113.165 137.125) (width 0.5) (layer F.Cu) (net 75))
@@
   (segment (start 187.4 161.515) (end 187.315 161.6) (width 0.5) (layer F.Cu) (net 76))
   (segment (start 187.4 160.35) (end 187.4 161.515) (width 0.5) (layer F.Cu) (net 76))
-  (segment (start 182.785 161.665) (end 183.8 160.65) (width 0.5) (layer F.Cu) (net 77))
-  (segment (start 182.785 162.15) (end 182.785 161.665) (width 0.5) (layer F.Cu) (net 77))
-  (segment (start 184.75 159.7) (end 183.8 160.65) (width 0.5) (layer F.Cu) (net 77))
-  (segment (start 185.4 159.7) (end 184.75 159.7) (width 0.5) (layer F.Cu) (net 77))
+  (segment (start 181.85 158.75) (end 182.8 159.7) (width 0.3) (layer F.Cu) (net 77))
+  (segment (start 181.8 158.75) (end 181.85 158.75) (width 0.3) (layer F.Cu) (net 77))
+  (segment (start 182.8 159.7) (end 182.785 159.715) (width 0.3) (layer F.Cu) (net 77))
+  (segment (start 185.4 160.225) (end 185.4 159.7) (width 0.3) (layer F.Cu) (net 77))
+  (segment (start 182.785 159.715) (end 182.785 160.585) (width 0.3) (layer F.Cu) (net 77))
+  (segment (start 182.785 160.585) (end 182.985 160.585) (width 0.3) (layer F.Cu) (net 77))
+  (segment (start 182.785 160.585) (end 182.785 162.15) (width 0.3) (layer F.Cu) (net 77))
+  (segment (start 185.025 160.6) (end 185.4 160.225) (width 0.3) (layer F.Cu) (net 77))
+  (segment (start 183 160.6) (end 185.025 160.6) (width 0.3) (layer F.Cu) (net 77))
+  (segment (start 182.985 160.585) (end 183 160.6) (width 0.3) (layer F.Cu) (net 77))
   (segment (start 116.415 104.9) (end 116.2 105.115) (width 0.5) (layer F.Cu) (net 78))
   (segment (start 116.415 103.4) (end 116.415 104.9) (width 0.5) (layer F.Cu) (net 78))

Commit message: update : sch
Parts:
- removed C10, C9: 1u, Capacitor_SMD:C_0603_1608Metric
- removed C23: 22u, Capacitor_SMD:C_0805_2012Metric
- removed D1: D_Schottky, Diode_SMD:D_SOD-123F
- removed D3: LED, LED_SMD:LED_0603_1608Metric
- removed J1: USB_C_Receptacle_USB2.0, Connector_USB:USB_C_Receptacle_GCT_USB4085
- removed J13, J14: Conn_01x04, Connector_JST:JST_XH_B4B-XH-A_1x04_P2.50mm_Vertical
- removed Q1: 2SC4116, Package_TO_SOT_SMD:SOT-323_SC-70
- removed Q3: IRLML6402, Package_TO_SOT_SMD:SOT-23
- removed R11, R13, R9: 10k, Resistor_SMD:R_0402_1005Metric
- removed R15: 1k, Resistor_SMD:R_0402_1005Metric
- removed R17, R18, R20, R21: 2k, Resistor_SMD:R_0402_1005Metric
- removed R2: 5.1k, Resistor_SMD:R_0402_1005Metric
- removed R5, R6, R7: 0 N.C., Resistor_SMD:R_0402_1005Metric
- added SW1: SW_SPST, Button_Switch_SMD:SW_Push_1P1T_NO_CK_KMR2, F.Cu at (126.3, 141.2)
- C4: value 22u -> 0.1u; footprint Capacitor_SMD:C_0805_2012Metric -> Capacitor_SMD:C_0402_1005Metric
- R1: value 5.1k -> 10k
- moved R1 24.6 mm to (127.0, 136.4), turned to 90 degrees
- moved H3 20.0 mm to (176.0, 104.0)
- moved H4 20.0 mm to (176.0, 186.0)
- moved J10 19.5 mm to (171.7, 140.4)
- moved J12 19.5 mm to (171.7, 133.6)
- moved J6 19.5 mm to (171.7, 154.0)
- moved J8 19.5 mm to (171.7, 147.2)
- moved D13 19.0 mm to (175.1, 168.9)
- moved D14 19.0 mm to (175.1, 166.3)
- moved D15 19.0 mm to (175.1, 163.7)
- moved J11 19.0 mm to (160.6, 133.6)
- moved J5 19.0 mm to (160.6, 154.0)
- moved J7 19.0 mm to (160.6, 147.2)
- moved J9 19.0 mm to (160.6, 140.4)
- moved R38 19.0 mm to (178.3, 168.9)
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Connections:
- C4 pad 1: +5VP -> +3V3
- C4 pad 2: GND -> /USER_SWITCH
- C6 pad 1: VBUS -> +5VP
- D2 pad 2: VBUS -> +5VP
- D5 pad 1: VBUS -> +5VP
- R1 pad 1: Net-(J1-PadA5) -> GND
- R1 pad 2: GND -> /USER_SWITCH
- R4 pad 1: VBUS -> VCC
- U1 pad 11: /ENC_PWR -> Net-(U1-Pad11)
- U1 pad 16: Net-(U1-Pad16) -> /USER_SWITCH
- U1 pad 4: /ENC1_A -> Net-(U1-Pad4)
- U1 pad 48: Net-(U1-Pad48) -> VCC
- U1 pad 49: VCC -> Net-(U1-Pad49)
- U1 pad 5: /ENC1_B -> Net-(U1-Pad5)
- U1 pad 6: /ENC2_A -> Net-(U1-Pad6)
- U1 pad 7: /ENC2_B -> Net-(U1-Pad7)
- U2 pad 3: VBUS -> +5VP
Routing:
- net +3.3VP: track 205.5 -> 0.00 mm, vias 13 -> 0
- net +5VP: track 139.3 -> 0.00 mm, vias 5 -> 0
- net /5V_P3: track 97.4 -> 0.00 mm
- net /CAN1_RX: track 71.6 -> 0.00 mm, vias 1 -> 0
- net /CAN1_TX: track 70.9 -> 0.00 mm, vias 1 -> 0
- net /CAN2_RX: track 69.6 -> 0.00 mm, vias 2 -> 0
- net /CAN2_TX: track 65.7 -> 0.00 mm, vias 2 -> 0
- net /WALL_VCC: track 64.0 -> 0.00 mm
- net /SERIAL2_EN: track 61.3 -> 0.00 mm
- net /ENC2_A: track 58.1 -> 0.00 mm
- net /VCC_P3-2: track 57.6 -> 0.00 mm
- net +5VL: track 56.1 -> 0.00 mm, vias 2 -> 0
- net /ENC1_A: track 55.9 -> 0.00 mm
- net /ENC2_B: track 53.0 -> 0.00 mm
- net /ENC1_B: track 52.7 -> 0.00 mm
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- removed copper zone on B.Cu, net +3.3VP
- removed copper zone on F.Cu, net +3.3VP
- removed copper zone on B.Cu, net /GND_P1
- removed copper zone on F.Cu, net /GND_P1
- removed copper zone on B.Cu, net /GND_P3
- removed copper zone on F.Cu, net /GND_P3
- removed copper zone on B.Cu, net /VCC_P3
- removed copper zone on B.Cu, net GND
- removed copper zone on F.Cu, net GND
Other:
- board size 100 x 90 mm -> 80 x 90 mm
- board text added: "FMSKF RobotController V1.1"
- board text added: "Sts1"
- board text added: "Sts2"
- board text added: "Sts3"
- board text removed: "ENC1"
- board text removed: "ENC2"
- board text removed: "EncPwr"
- board text removed: "Ext 5VL"
- board text removed: "Ext 5VP"
- board text removed: "FMSKF RobotContoller V1"
- board text removed: "Status1"
- board text removed: "Status2"
- board text removed: "Status3"
- board text removed: "Tnsy Cn Ext"

Commit message: board update v2
Parts:
- removed J23: Conn_02x03_Odd_Even, Connector_PinHeader_2.00mm:PinHeader_2x03_P2.00mm_Vertical
- removed R19: 0 N.C., Resistor_SMD:R_0402_1005Metric
- removed R4, R8: 0, Resistor_SMD:R_0402_1005Metric
- added D1: PMEG6010CEGWJ, Diode_SMD:D_SOD-123, F.Cu at (114.4, 105.9)
- added J1: USB_C_Receptacle_USB2.0, Connector_USB:USB_C_Receptacle_GCT_USB4085, F.Cu at (125.2, 109.0)
- added R2: 5.1k, Resistor_SMD:R_0402_1005Metric, F.Cu at (123.5, 111.4)
- added R5: 5.1k, Resistor_SMD:R_0402_1005Metric, F.Cu at (114.4, 102.0)
- U1: value Teensy4.1_simple -> Teensy4.1; footprint teensy_FP:Teensy41simple -> teensy_FP:Teensy41_onlyeth
- moved C4 13.2 mm to (125.4, 149.6), turned to 0 degrees
- moved SW1 12.4 mm to (125.4, 153.6)
- moved R1 12.1 mm to (125.4, 148.4), turned to 0 degrees
- moved C6 8.91 mm to (113.6, 110.6)
- moved D5 7.96 mm to (118.3, 113.5)
- moved U2 7.96 mm to (112.1, 115.5)
- moved C7 7.96 mm to (117.7, 116.7)
- moved C8 7.96 mm to (119.2, 116.7)
- moved D2 4.75 mm to (105.6, 115.5)
- moved D6 4.75 mm to (105.6, 118.0)
- moved R22 4.75 mm to (102.7, 118.0)
- moved R3 4.75 mm to (102.7, 115.5)
- moved R36 3.32 mm to (111.1, 151.9), turned to 270 degrees
- moved D12 2.92 mm to (114.3, 176.8)
- moved D4 2.11 mm to (174.1, 159.9)
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Connections:
- C24 pad 1: +5VP -> +5VL
- C5 pad 1: +5VP -> +5VL
- C6 pad 1: +5VP -> +5VL
- D2 pad 2: +5VP -> +5VL
- D5 pad 1: +5VP -> +5VL
- Q4 pad 2: +5VP -> +5VL
- R12 pad 1: +5VP -> +5VL
- U1 pad 48: VCC -> +5VL
- U2 pad 3: +5VP -> +5VL
Routing:
- net +5VL: track 0.00 -> 185.3 mm, vias 0 -> 4
- net +3.3VP: track 0.00 -> 152.5 mm, vias 0 -> 12
- net /5V_P3: track 0.00 -> 78.5 mm, vias 0 -> 2
- net /CAN1_RX: track 0.00 -> 78.4 mm
- net /CAN1_TX: track 0.00 -> 77.6 mm, vias 0 -> 2
- net /CAN2_TX: track 0.00 -> 73.4 mm
- net /CAN2_RX: track 0.00 -> 65.3 mm
- net /WALL_VCC: track 0.00 -> 63.2 mm
- net /VCC_P3-2: track 0.00 -> 46.5 mm
- net /IMU_SPI_CS1: track 0.00 -> 45.6 mm, vias 0 -> 3
- net /IMU_SPI_CS2: track 0.00 -> 43.7 mm, vias 0 -> 3
- net /SERIAL2_EN: track 0.00 -> 43.0 mm, vias 0 -> 2
- net /WALL_AD1: track 0.00 -> 42.7 mm
- net /WALL_AD3: track 0.00 -> 39.7 mm
- net /WALL_AD5: track 0.00 -> 37.2 mm
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- added copper zone on B.Cu, net +3.3VP
- added copper zone on F.Cu, net +3.3VP
- added copper zone on B.Cu, net +5VL
- added copper zone on F.Cu, net +5VL
- added copper zone on B.Cu, net /GND_P1
- added copper zone on F.Cu, net /GND_P1
- added copper zone on B.Cu, net /GND_P3
- added copper zone on F.Cu, net /GND_P3
- added copper zone on B.Cu, net /VCC_P3
- added copper zone on B.Cu, net GND
- added copper zone on F.Cu, net GND
Other:
- board text removed: "Tnsy 5VL"
- board text removed: "Tnsy 5VP"

Commit message: sch update
Parts:
- removed J22: Conn_01x02, Connector_JST:JST_EH_S2B-EH_1x02_P2.50mm_Horizontal
- removed R32, R34: 0, Resistor_SMD:R_0402_1005Metric
- added IC6: TLT9251VLEXUMA1, SamacSys_Parts:SON65P300X300X110-9N, F.Cu at (168.6, 167.0)
- added J13: Conn_01x04, Connector_JST:JST_EH_S4B-EH_1x04_P2.50mm_Horizontal, F.Cu at (173.0, 169.7)
- added R4: 0, Resistor_SMD:R_0402_1005Metric, F.Cu at (165.4, 165.9)
- added R6: 0, Resistor_SMD:R_0402_1005Metric, F.Cu at (165.4, 168.1)
- added R7: 60, Resistor_SMD:R_0402_1005Metric, F.Cu at (170.3, 171.2)
- added R8: 0, Resistor_SMD:R_0402_1005Metric, F.Cu at (141.8, 165.1)
- added R9: 0, Resistor_SMD:R_0402_1005Metric, F.Cu at (140.5, 165.1)
- IC1, IC2, IC5: value ADM3058EBRIZ-RL -> ISO1044BDR; footprint SamacSys_Parts:SOIC127P1031X265-8N -> SamacSys_Parts:SOIC127P600X175-8N
- U1: footprint teensy_FP:Teensy41_onlyeth -> teensy_FP:Teensy41simple_onlyeth
- moved IC1 25.2 mm to (141.1, 172.6)
- moved IC5 22.5 mm to (164.9, 173.1)
- moved R38 4.80 mm to (176.9, 164.3)
- moved D13 4.61 mm to (174.1, 164.4)
- moved R39 4.04 mm to (176.9, 162.5)
- moved D14 3.93 mm to (174.1, 162.5)
- moved R40 3.31 mm to (176.9, 160.7)
- moved D15 3.16 mm to (174.1, 160.7)
- moved C15 2.69 mm to (168.3, 175.0)
- moved C11 2.28 mm to (168.3, 171.2)
- moved C20 2.23 mm to (144.5, 175.9), turned to 270 degrees
- moved C18 1.80 mm to (145.0, 168.2)
- moved IC2 1.20 mm to (128.8, 172.7)
- moved C16 1.15 mm to (132.2, 176.0), turned to 270 degrees
- moved R16 1.00 mm to (176.9, 158.9)
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Connections:
- IC1 pad 2: /CAN1_TX -> Net-(IC1-Pad2)
- IC1 pad 3: /CAN1_RX -> Net-(IC1-Pad3)
- IC1 pad 5: /GND_P1 -> /CAN2_L
- IC1 pad 6: /CAN1_L -> /CAN2_H
- IC1 pad 7: /CAN1_H -> /GND_P3
- IC1 pad 8: /5V_P1 -> /5V_P3
- IC2 pad 5: /GND_P3 -> /CAN3_L
- IC2 pad 6: /CAN3_L -> /CAN3_H
- IC2 pad 7: /CAN3_H -> /GND_P3
- IC5 pad 2: /CAN2_TX -> /CAN1_TX
- IC5 pad 3: /CAN2_RX -> /CAN1_RX
- IC5 pad 5: /GND_P3 -> /CAN1_L
- IC5 pad 6: /CAN2_L -> /CAN1_H
- IC5 pad 7: /CAN2_H -> /GND_P1
- IC5 pad 8: /5V_P3 -> /5V_P1
- J21 pad 2: /VCC_P3-2 -> /VCC_P3
- U1 pad 17: Net-(U1-Pad17) -> /IMU_SPI_CS1
- U1 pad 18: Net-(U1-Pad18) -> /IMU_SPI_CS2
- U1 pad 28: /IMU_SPI_CS2 -> Net-(U1-Pad28)
- U1 pad 29: /IMU_SPI_CS1 -> Net-(U1-Pad29)
- U1 pad 32: Net-(U1-Pad32) -> /WALLTOF_CAN_EN
Routing:
- net /VCC_P3: track 24.8 -> 77.7 mm
- net /VCC_P3-2: track 46.5 -> 0.00 mm
- net /WALLTOF_CAN_EN: track 0.00 -> 39.9 mm, vias 0 -> 2
- net /CAN2_RX: track 65.3 -> 90.2 mm, vias 0 -> 2
- net +5VL: track 185.3 -> 208.1 mm
- net /WALL_VCC: track 63.2 -> 85.3 mm
- net /CAN2_TX: track 73.4 -> 94.5 mm, vias 0 -> 2
- net /IMU_SPI_CS1: track 45.6 -> 29.1 mm, vias 3 -> 2
- net /IMU_SPI_CS2: track 43.7 -> 31.5 mm, vias 3 -> 1
- net +3.3VP: track 152.5 -> 162.4 mm, vias 12 -> 13
- net Net-(IC6-Pad6): track 0.00 -> 9.16 mm
- net Net-(IC6-Pad7): track 0.00 -> 8.91 mm
- net /CAN1_RX: track 78.4 -> 85.5 mm
- net /CAN1_TX: track 77.6 -> 84.0 mm, vias 2 -> 0
- net /5V_P3: track 78.5 -> 72.9 mm
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Other:
- board text added: "GVLH"
